Commit message: feat: Added models to environment

File: src/ur_robotiq_description/urdf/ur_robotiq.urdf.xacro (robot description, xacro)
@@ -94,5 +94,5 @@
      trajectory_port="$(arg trajectory_port)"
      >
-    <origin xyz="0 0 0" rpy="0 0 0" />          <!-- position robot in the world -->
+    <origin xyz="-1.3 0.2 1.5" rpy="-1.57079632679 -1.57079632679 -1.57079632679" />          <!-- position robot in the world -->
     </xacro:ur_robot>
    <xacro:robotiq_gripper name="$(arg tf_prefix)gripper"

Commit message: feat: added collision for moveit

File: src/ur_robotiq_description/urdf/ur_robotiq.urdf.xacro (robot description, xacro)
@@ -94,5 +94,5 @@
      trajectory_port="$(arg trajectory_port)"
      >
-    <origin xyz="-1.3 0.2 1.5" rpy="-1.57079632679 -1.57079632679 -1.57079632679" />          <!-- position robot in the world -->
+    <origin xyz="-1.3 0.2 1.5" rpy="0 -1.57079632679 -1.57079632679" />          <!-- position robot in the world -->
     </xacro:ur_robot>
    <xacro:robotiq_gripper name="$(arg tf_prefix)gripper"

File: src/ur_robotiq_moveit_config/srdf/ur_robotiq_macro.srdf.xacro (robot description, xacro)
@@ -40,9 +40,9 @@
     </group_state>
     <group_state name="${prefix}home" group="${prefix}${name}_manipulator">
-      <joint name="${prefix}elbow_joint" value="0" />
-      <joint name="${prefix}shoulder_lift_joint" value="-1.5707" />
+      <joint name="${prefix}elbow_joint" value="-0.837758" />
+      <joint name="${prefix}shoulder_lift_joint" value="-1.22173" />
       <joint name="${prefix}shoulder_pan_joint" value="0" />
-      <joint name="${prefix}wrist_1_joint" value="0" />
-      <joint name="${prefix}wrist_2_joint" value="0" />
+      <joint name="${prefix}wrist_1_joint" value="-1.06465" />
+      <joint name="${prefix}wrist_2_joint" value="1.5708" />
       <joint name="${prefix}wrist_3_joint" value="0" />
     </group_state>

Commit message: feat:add tcp and improved tf

File: src/ur_robotiq_description/urdf/ur_robotiq.urdf.xacro (robot description, xacro)
@@ -104,3 +104,10 @@
     <origin xyz="0 0 0" rpy="0 0 0" />
     </xacro:robotiq_gripper>
+   <!-- Canonical grasp/TCP frame between gripper fingertips. -->
+   <link name="$(arg tf_prefix)TCP_point"/>
+   <joint name="$(arg tf_prefix)tool0_tcp_point_joint" type="fixed">
+     <parent link="$(arg tf_prefix)tool0"/>
+     <child link="$(arg tf_prefix)TCP_point"/>
+     <origin xyz="0 0 0.2" rpy="0 0 0"/>
+   </joint>
 </robot>

File: src/ur_robotiq_moveit_config/srdf/ur_robotiq_macro.srdf.xacro (robot description, xacro)
@@ -12,5 +12,5 @@
     <!--SUBGROUPS Groups can also be formed by referencing to already defined group names-->
     <group name="${prefix}${name}_manipulator">
-        <chain base_link="${prefix}base_link" tip_link="${prefix}tool0"/>
+        <chain base_link="${prefix}base_link" tip_link="${prefix}TCP_point"/>
     </group>
     <group name="${prefix}gripper">
@@ -64,5 +64,5 @@
     </group_state>
     <!--END EFFECTOR Purpose Represent information about an end effector.-->
-    <end_effector name="${prefix}gripper" parent_link="${prefix}tool0" group="${prefix}gripper" parent_group="${prefix}${name}_manipulator"/>
+    <end_effector name="${prefix}gripper" parent_link="${prefix}TCP_point" group="${prefix}gripper" parent_group="${prefix}${name}_manipulator"/>
     <!--VIRTUAL JOINT Purpose this element defines a virtual joint between a robot link and an external frame of reference (considered fixed with respect to the robot)-->
     <virtual_joint name="world_joint" type="fixed" parent_frame="world" child_link="${prefix}base_link"/>
