Commit message: feat: Added support for the curobo mpc method

File: src/ur_robotiq_description/urdf/ur_gantry_7dof.urdf (robot description, URDF)
Before this commit: robot ur_gantry, 29 links, 28 joints
Joints:
- joint gantry_joint: limit lower=-0.75 upper=0.75 effort=2000.0 velocity=0.8 -> lower=-0.75 upper=0.75 effort=2000.0 velocity=1.0

File: src/ur_robotiq_description/urdf/ur_gantry_7dof_no_gripper.urdf (robot description, URDF)
Before this commit: robot ur_gantry, 17 links, 16 joints
Joints:
- joint gantry_joint: limit lower=-0.75 upper=0.75 effort=2000.0 velocity=0.8 -> lower=-0.75 upper=0.75 effort=2000.0 velocity=1.0

File: src/ur_robotiq_description/urdf/ur_robotiq_gantry.urdf.xacro (robot description, xacro)
@@ -55,5 +55,5 @@
   <xacro:arg name="gantry_lower_limit" default="-0.75"/>
   <xacro:arg name="gantry_upper_limit" default="0.75"/>
-  <xacro:arg name="gantry_velocity_limit" default="0.8"/>
+  <xacro:arg name="gantry_velocity_limit" default="1.0"/>
   <xacro:arg name="gantry_effort_limit" default="2000.0"/>
   <xacro:arg name="gantry_beam_length" default="3.0"/>
