Commit message: feat: pick and place pipeline

File: src/ros2_robotiq_gripper/robotiq_description/urdf/robotiq_2f_140.xacro (robot description, xacro)
@@ -136,5 +136,5 @@
         <origin xyz="0 0 0" rpy="0 0 0" />
         <geometry>
-           <box size="0.03 0.07 0.0075"/>
+           <box size="0.027 0.07 0.0075"/>
         </geometry>
         <material name="">

File: src/ur_robotiq_description/urdf/ur_robotiq.urdf.xacro (robot description, xacro)
@@ -109,5 +109,5 @@
      <parent link="$(arg tf_prefix)tool0"/>
      <child link="$(arg tf_prefix)TCP_point"/>
-     <origin xyz="0 0 0.2" rpy="0 0 0"/>
+     <origin xyz="0 0 0.21" rpy="0 0 0"/>
    </joint>
 </robot>
