Commit message: feat: added 7dof while still keeping 6 dof as backup

File: src/Universal_Robots_ROS2_Description/urdf/isaac_ur.ros2_control.xacro (robot description, xacro)
@@ -7,8 +7,9 @@
     sim_ignition:=false
     sim_isaac:=false
+    enable_gantry:=false
     isaac_joint_commands:=/isaac_joint_commands
     isaac_joint_states:=/joint_states
     headless_mode:=false
-    initial_positions:=${dict(shoulder_pan_joint=0.0,shoulder_lift_joint=-1.57,elbow_joint=0.0,wrist_1_joint=-1.57,wrist_2_joint=0.0,wrist_3_joint=0.0)}
+    initial_positions:=${dict(gantry_joint=0.0,shoulder_pan_joint=0.0,shoulder_lift_joint=-1.57,elbow_joint=0.0,wrist_1_joint=-1.57,wrist_2_joint=0.0,wrist_3_joint=0.0)}
     use_tool_communication:=false
     script_filename output_recipe_filename
@@ -28,9 +29,16 @@
     <hardware>
       <plugin>topic_based_ros2_control/TopicBasedSystem</plugin>
-      <param name="joint_commands_topic">/isaac_joint_commands</param>
-      <param name="joint_states_topic">/joint_states</param>
+      <param name="joint_commands_topic">${isaac_joint_commands}</param>
+      <param name="joint_states_topic">${isaac_joint_states}</param>
       <param name="trigger_joint_command_threshold">-1</param>
     </hardware>
-    <!-- Ajouter ici uniquement les joints actifs -->
+    <!-- Active joints for topic-based ros2_control -->
+    <xacro:if value="${enable_gantry}">
+      <joint name="gantry_joint">
+        <command_interface name="position"/>
+        <state_interface name="position"/>
+        <state_interface name="velocity"/>
+      </joint>
+    </xacro:if>
     <joint name="shoulder_pan_joint">
       <command_interface name="position"/>

File: src/Universal_Robots_ROS2_Description/urdf/ur.ros2_control.xacro (robot description, xacro)
@@ -7,8 +7,9 @@
     sim_ignition:=false
     sim_isaac:=false
+    enable_gantry:=false
     isaac_joint_commands:=/isaac_joint_commands_ur
     isaac_joint_states:=/joint_states
     headless_mode:=false
-    initial_positions:=${dict(shoulder_pan_joint=0.0,shoulder_lift_joint=-1.57,elbow_joint=0.0,wrist_1_joint=-1.57,wrist_2_joint=0.0,wrist_3_joint=0.0)}
+    initial_positions:=${dict(gantry_joint=0.0,shoulder_pan_joint=0.0,shoulder_lift_joint=-1.57,elbow_joint=0.0,wrist_1_joint=-1.57,wrist_2_joint=0.0,wrist_3_joint=0.0)}
     use_tool_communication:=false
     script_filename output_recipe_filename
@@ -73,4 +74,16 @@
         </xacro:unless>
       </hardware>
+      <xacro:if value="${enable_gantry}">
+        <joint name="${tf_prefix}gantry_joint">
+          <command_interface name="position"/>
+          <command_interface name="velocity"/>
+          <state_interface name="position">
+            <!-- initial position for the FakeSystem and simulation -->
+            <param name="initial_value">${initial_positions['gantry_joint']}</param>
+          </state_interface>
+          <state_interface name="velocity"/>
+          <state_interface name="effort"/>
+        </joint>
+      </xacro:if>
       <joint name="${tf_prefix}shoulder_pan_joint">
         <command_interface name="position"/>

File: src/Universal_Robots_ROS2_Description/urdf/ur_macro.xacro (robot description, xacro)
@@ -55,4 +55,5 @@
     generate_ros2_control_tag:=true
     sim_isaac:=false
+    enable_gantry:=false
     isaac_joint_commands:=/isaac_joint_commands
     isaac_joint_states:=/joint_states
@@ -112,4 +113,5 @@
         sim_ignition="${sim_ignition}"
         sim_isaac="${sim_isaac}"
+        enable_gantry="${enable_gantry}"
         isaac_joint_commands="${isaac_joint_commands}"
         isaac_joint_states="${isaac_joint_states}"

File: src/ros2_robotiq_gripper/robotiq_description/urdf/2f_140.ros2_control.xacro (robot description, xacro)
@@ -6,5 +6,5 @@
         sim_gazebo:=false
         sim_isaac:=false
-        isaac_joint_commands:=/isaac_joint_commands_robotiq
+        isaac_joint_commands:=/isaac_joint_gripper
         isaac_joint_states:=/joint_states
         use_fake_hardware:=false
@@ -16,4 +16,8 @@
         gripper_max_force:=125.0
         gripper_closed_position:=0.695">
+        <xacro:property name="finger_joint_initial_value" value="${gripper_closed_position}"/>
+        <xacro:if value="${sim_isaac}">
+            <xacro:property name="finger_joint_initial_value" value="0.0"/>
+        </xacro:if>
         <ros2_control name="${name}" type="system">
             <!-- Plugins -->
@@ -21,5 +25,5 @@
                 <xacro:if value="${sim_isaac}">
                     <plugin>topic_based_ros2_control/TopicBasedSystem</plugin>
-                    <param name="joint_commands_topic">/isaac_joint_gripper</param>
+                    <param name="joint_commands_topic">${isaac_joint_commands}</param>
                     <param name="joint_states_topic">${isaac_joint_states}</param>
                     <param name="trigger_joint_command_threshold">-1</param>
@@ -48,5 +52,5 @@
                 <command_interface name="position" />
                 <state_interface name="position">
-                    <param name="initial_value">${gripper_closed_position}</param>
+                    <param name="initial_value">${finger_joint_initial_value}</param>
                 </state_interface>
                 <state_interface name="velocity"/>

File: src/ros2_robotiq_gripper/robotiq_description/urdf/robotiq_2f_140.xacro (robot description, xacro)
@@ -170,5 +170,4 @@
       <parent link="${prefix}${fingerprefix}_outer_knuckle" />
       <child link="${prefix}${fingerprefix}_outer_finger" />
-      <axis xyz="1 0 0" />
     </joint>
   </xacro:macro>
@@ -198,5 +197,4 @@
       <parent link="${prefix}${fingerprefix}_inner_finger" />
       <child link="${prefix}${fingerprefix}_inner_finger_pad" />
-      <axis xyz="0 0 1" />
     </joint>
   </xacro:macro>

File: src/ur_robotiq_description/urdf/ur_robotiq.urdf.xacro (robot description, xacro)
@@ -48,4 +48,5 @@
 	<xacro:arg name="sim_isaac" default="false" />
 	<xacro:arg name="isaac_joint_commands" default="/isaac_joint_commands" />
+	<xacro:arg name="isaac_gripper_joint_commands" default="/isaac_joint_gripper" />
 	<xacro:arg name="isaac_joint_states" default="/joint_states" />
 	<!-- initial position for simulations (Fake Hardware, Gazebo, Ignition) -->
@@ -101,4 +102,6 @@
     use_fake_hardware="$(arg use_fake_hardware)"
     sim_isaac="$(arg sim_isaac)"
+    isaac_joint_commands="$(arg isaac_gripper_joint_commands)"
+    isaac_joint_states="$(arg isaac_joint_states)"
     >
     <origin xyz="0 0 0" rpy="0 0 0" />
